File: g3d2_ctrl_2.brd (EAGLE design)
At the start: 80 x 80 mm, 44 parts, among them IC1 atmega88pa, IC10 78L05SMD, IC11 LT3972, IC2 IRF7103, IC3 IRF7103, IC4 IRF7103, IC5 IRF7103, IC6 IRF7104, IC7 IRF7104, IC8 IRF7104, IC9 IRF7104, Q1 20Mhz

Commit message: production ready
Parts:
- moved JP1 1.40 mm to (33.5, 8.21)
- moved JP2 1.40 mm to (8.15, 31.2)
- moved JP4 0.90 mm to (18.2, 83.0)
- moved JP3 0.80 mm to (82.9, 46.5)
Routing:
- net +12V: track 317.9 -> 310.3 mm
- net GND: track 70.1 -> 76.8 mm
- net RX: track 222.6 -> 225.4 mm
- net TX: track 207.1 -> 207.2 mm, vias 3 -> 7
Other:
- outline, holes or cut-outs redrawn
